File: KiCad/led-controller.kicad_pcb (KiCad board)
At the start: 2 copper layers, 96.5 x 36.8 mm, 25 parts, among them J1 Conn_01x02_Male, J2 Conn_01x03_Male, J3 Conn_01x04_Male, Q1 BSS138, SW1 FLASH, SW2 RESET, U1 Meanwell_MPM-20-5, U2 AMS1117-3.3, U3 ESP8266-12E/ESP-12E

Commit message: roses are red, plus is minus and i fucked up
Routing:
- net Net-(R6-Pad1): track 49.6 -> 17.5 mm, vias 0 -> 2
- net Net-(R1-Pad2): track 33.6 -> 23.6 mm
- net Net-(J2-Pad2): track 83.1 -> 80.3 mm, vias 2 -> 1
- net +3V3: track 133.6 -> 132.2 mm
- net Net-(Q1-Pad2): track 32.0 -> 32.9 mm, vias 0 -> 3
- net +5V: track 108.7 -> 107.9 mm, vias 1 -> 0
- net GND: vias 3 -> 2
